Commit message: LICENSE

File: Inverse kinematics full along with manual control/my_robot/robot.urdf (robot description, URDF)
Before this commit: robot D:\ArMigo(Camera detection)\my-robot, 7 links, 6 joints
Links:
- link base: geometry collision mesh filename=package://assets/base.stl; collision mesh filename=package://assets/base_cover.stl
- link base_joint: geometry collision mesh filename=package://assets/base_joint.stl; visual mesh filename=package://assets/base_joint.stl
- link elbow: geometry collision mesh filename=package://assets/joint_2.stl; visual mesh filename=package://assets/joint_2.stl
- link gripper: geometry collision mesh filename=package://assets/part_1.stl; collision mesh filename=package://assets/part_2.stl
- link joint_4: geometry collision mesh filename=package://assets/joint_4.stl; visual mesh filename=package://assets/joint_4.stl
- link shoulders: geometry collision mesh filename=package://assets/joint_1.stl; collision mesh filename=package://assets/joint_1__cover.stl
